File: hardware/base/kicad/base.kicad_pcb (KiCad board)
At the start: 4 copper layers, 150 x 72 mm, 525 parts, among them J1 POWER, J10 LOCAL BUS, J11 SPINDLE A, J12 SPINDLE B, J13 MODBUS, J14 ESTOP | PROBE, J2 USB micro-B, J3 HY911105AE IN, J4 HY911105AE OUT, J5 TC2030, J6 HC-WK88-H132-1X2-55B, J7 HC-WK88-H132-1X2-55B, J8 HC-WK88-H132-1X2-55B, J9 HC-WK88-H132-1X2-55B, Q1 AO3422, Q11 AO3401A, Q2 AO3422, Q3 AO3422, Q4 AO3422, Q5 SS8550, Q6 AO3422, Q7 AO3422, SW1 BOOT, U1 TPS54360BDDAR, U10 TPS1H000AQDGNRQ1, U11 ST26C31BDR, U12 LTV-357T-C, U13 TPD4E05U06DQAR, U14 LTV-357T-C, U15 TPD4E05U06DQAR, U16 ST26C31BDR, U17 LTV-357T-C, U18 TPD4E05U06DQAR, U19 LTV-357T-C, U2 TPD4E05U06DQAR, U20 TPD4E05U06DQAR, U21 TPS1H000AQDGNRQ1, U22 AM26LV32EIDR, U23 TPS1H000AQDGNRQ1, U24 AM26LV32EIDR, U25 TPS1H000AQDGNRQ1, U26 AM26LV32EIDR, U27 TPS1H000AQDGNRQ1, U28 AM26LV32EIDR, U29 TLP2361, U3 TPS62A02ADRLR, U30 TPS2553DBVR, U31 TPD4E05U06DQAR, U32 TPD4E05U06DQAR, U33 TPD4E05U06DQAR, U34 TPD4E05U06DQAR, U35 TPD4E05U06DQAR, U36 OPA2990IDR, U37 SN74AHCT1G125DBVR, U38 CA-IS3092W, U39 LTV-357T-C, U4 LAN9253-I/R4X, U40 TPS3828-33DBVR, U5 TPS3808G33DBVR, U6 M24C16-RMN6TP, U7 TPD4E05U06DQAR, U8 TPD4E05U06DQAR, U9 STM32H523VET6, X1 SiT8008BI-71-33E-25.000000

Commit message: Widen the base board to 107.5 x 150 mm, vertical USB, PE contact hole
- The parts covered 94 % of the free top area on 72 mm, 53 % on 107.5 mm:
  Phoenix UM-BASIC 108 profile (kit UM-BASIC-KIT-B108-L150-7035), one side.
- M3 holes at the four corners; H1 plated next to POWER.
- H5: plated hole for the Phoenix PE contact L1, which earths CHASSIS to
  the DIN rail; no lead over the contact body under the board.
- USB jack: vertical Molex 105133-0001, to sit next to the MCU.
Parts:
- added H5: PE CONTACT, MountingHole:MountingHole_3.2mm_M3_Pad, F.Cu at (143.9, 84.0)
- J2: footprint Connector_USB:USB_Micro-B_Amphenol_10118194-0001LF_Horizontal -> Connector_USB:USB_Micro-B_Molex-105133-0001
- moved R10 312.1 mm to (170.0, 45.0)
- moved R136 312.1 mm to (170.0, 53.0)
- moved R172 312.1 mm to (170.0, 61.0)
- moved R208 312.1 mm to (170.0, 69.0)
- moved R244 312.1 mm to (170.0, 77.0)
- moved R43 312.1 mm to (170.0, 85.0)
- moved R80 312.1 mm to (170.0, 93.0)
- moved U2 312.1 mm to (170.0, 101.0)
- moved J2 204.2 mm to (250.0, 37.0)
- moved H3 151.1 mm to (4.50, 4.50)
- moved H4 139.4 mm to (145.5, 4.50)
- moved H1 97.2 mm to (145.5, 103.0)
- moved H2 57.0 mm to (4.50, 103.0)
- moved J1 35.9 mm to (127.1, 99.0)
- moved J14 35.9 mm to (108.3, 99.0)
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Other:
- board size 150 x 72 mm -> 150 x 107.5 mm

Commit message: 3D models for every part of the base board; edge connectors flush
- gen_3d.py: simplified STEP models from the datasheets of the
  HY911105AE magjack, the Molex 105133-0001 vertical micro-B, the
  HX PZ2.54 SMD header and the TS-1187A switch.
- pcb.py: KiCad library footprints whose model is missing point to the
  same package under another name, or to a generated model.
- Edge connectors placed from their real front face, set back just enough
  for the pads of their front leads to clear the rim on the profile walls.
Parts:
- moved J3 2.59 mm to (13.4, 92.3)
- moved J4 2.59 mm to (33.5, 92.3)
- moved J6 0.35 mm to (25.5, 8.94)
- moved J7 0.35 mm to (58.5, 8.94)
- moved J8 0.35 mm to (91.5, 8.94)
- moved J9 0.35 mm to (124.5, 8.94)

Commit message: Place the base board parts; DIP switches for the encoder terminations
Placement (gen/pcb.py): one zone per schematic sheet, key parts placed by
hand, the other parts next to the pin they serve, bulkiest first, with a
1 mm gap preferred when it costs at most 2 mm. The local bus header stands
at the left end, centred across the board, facing the modules.

Encoder terminations: one CTS 218-4LPSTR DIP switch per encoder (100 mA
non-switching) replaces three SMD jumpers; the supply selector and the
Modbus termination use a through-hole 1x3 header. Split DIP symbol, one
unit per switch, drawn on the pair it serves.

DRC rules: 0.2 mm thermal vias, per-package clearance for 0.65 mm pitch
parts. Test points out of the BOM, DNP copied to the footprints. pcb.py
keeps the schematic settings of the project file and finds the KiCad
footprint libraries on every install.

Claude-Session: https://claude.ai/code/session_01JfmMsHNpEd1mfzHNWc4koJ
Parts:
- removed JP10, JP11, JP12, JP14, JP15, JP16, JP17, JP6, JP7, JP8: TERM, Bornier:PinHeader_1x03_P2.54mm_Vertical_SMD_HX_PZ254
- removed JP13, JP9: ENC 5V|VIN, Bornier:PinHeader_1x03_P2.54mm_Vertical_SMD_HX_PZ254
- added SW2: TERM A B Z, Button_Switch_SMD:SW_DIP_SPSTx04_Slide_KingTek_DSHP04TS_W7.62mm_P1.27mm, F.Cu at (24.6, 50.8)
- added SW3: TERM A B Z, Button_Switch_SMD:SW_DIP_SPSTx04_Slide_KingTek_DSHP04TS_W7.62mm_P1.27mm, F.Cu at (83.2, 36.9)
- added SW4: TERM A B Z, Button_Switch_SMD:SW_DIP_SPSTx04_Slide_KingTek_DSHP04TS_W7.62mm_P1.27mm, F.Cu at (112.5, 50.4)
- added SW5: TERM A B Z, Button_Switch_SMD:SW_DIP_SPSTx04_Slide_KingTek_DSHP04TS_W7.62mm_P1.27mm, F.Cu at (140.8, 45.8)
- JP1: footprint Bornier:PinHeader_1x03_P2.54mm_Vertical_SMD_HX_PZ254 -> Connector_PinHeader_2.54mm:PinHeader_1x03_P2.54mm_Vertical
- JP2, JP3, JP4: value TERM -> ENC 5V|VIN; footprint Bornier:PinHeader_1x03_P2.54mm_Vertical_SMD_HX_PZ254 -> Connector_PinHeader_2.54mm:PinHeader_1x03_P2.54mm_Vertical
- JP5: value ENC 5V|VIN -> TERM; footprint Bornier:PinHeader_1x03_P2.54mm_Vertical_SMD_HX_PZ254 -> Connector_PinHeader_2.54mm:PinHeader_1x03_P2.54mm_Vertical
- moved R207 464.2 mm to (17.8, 56.8), turned to 90 degrees
- moved C76 461.0 mm to (16.1, 66.0)
- moved R206 455.8 mm to (18.4, 46.7), turned to 180 degrees
- moved C75 454.5 mm to (15.6, 73.8)
- moved R205 448.2 mm to (17.9, 52.2), turned to 90 degrees
- moved D34 446.4 mm to (35.9, 35.5), turned to 180 degrees
- moved D33 443.4 mm to (30.7, 31.1), turned to -90 degrees
- moved R204 443.2 mm to (14.9, 53.4), turned to 90 degrees
- moved R42 441.2 mm to (41.0, 62.9)
- moved R40 440.3 mm to (26.0, 61.9)
- moved R17 438.6 mm to (28.2, 80.7), turned to -90 degrees
- moved C39 434.3 mm to (45.0, 72.4), turned to -90 degrees
- moved R203 432.3 mm to (17.9, 49.2), turned to 90 degrees
- moved D32 431.3 mm to (35.4, 45.0), turned to 180 degrees
- moved R41 431.1 mm to (43.0, 67.2), turned to 90 degrees
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Connections:
- JP2 pad 1: /Encoder 0/AP -> +5V
- JP2 pad 2: Net-(JP2-C) -> /Encoder 1/VSEL
- JP2 pad 3: unconnected-(JP2-B-Pad3) -> +VIN
- JP3 pad 1: /Encoder 0/BP -> +5V
- JP3 pad 2: Net-(JP3-C) -> /Encoder 2/VSEL
- JP3 pad 3: unconnected-(JP3-B-Pad3) -> +VIN
- JP4 pad 1: /Encoder 0/ZP -> +5V
- JP4 pad 2: Net-(JP4-C) -> /Encoder 3/VSEL
- JP4 pad 3: unconnected-(JP4-B-Pad3) -> +VIN
- JP5 pad 1: +5V -> Net-(JP5-A)
- JP5 pad 2: /Encoder 1/VSEL -> /Modbus/MB_B
- JP5 pad 3: +VIN -> unconnected-(JP5-B-Pad3)
- R105 pad 1: Net-(JP4-C) -> Net-(R105-Pad1)
- R246 pad 2: Net-(JP17-A) -> Net-(JP5-A)
- R89 pad 1: Net-(JP2-C) -> Net-(R89-Pad1)
- R97 pad 1: Net-(JP3-C) -> Net-(R97-Pad1)
