File: hardware/base/kicad/base.kicad_pcb (KiCad board)
At the start: 4 copper layers, 150 x 107.5 mm, 518 parts, among them J1 POWER, J10 LOCAL BUS, J11 SPINDLE A, J12 SPINDLE B, J13 MODBUS, J14 ESTOP | PROBE, J2 USB micro-B, J3 HY911105AE IN, J4 HY911105AE OUT, J5 TC2030, J6 HC-WK88-H132-1X2-55B, J7 HC-WK88-H132-1X2-55B, J8 HC-WK88-H132-1X2-55B, J9 HC-WK88-H132-1X2-55B, Q1 AO3422, Q11 AO3401A, Q2 AO3422, Q3 AO3422, Q4 AO3422, Q5 SS8550, Q6 AO3422, Q7 AO3422, SW1 BOOT, SW2 TERM A B Z, SW3 TERM A B Z, SW4 TERM A B Z, SW5 TERM A B Z, U1 TPS54360BDDAR, U10 TPS1H000AQDGNRQ1, U11 ST26C31BDR, U12 LTV-357T-C, U13 TPD4E05U06DQAR, U14 LTV-357T-C, U15 TPD4E05U06DQAR, U16 ST26C31BDR, U17 LTV-357T-C, U18 TPD4E05U06DQAR, U19 LTV-357T-C, U2 TPD4E05U06DQAR, U20 TPD4E05U06DQAR, U21 TPS1H000AQDGNRQ1, U22 AM26LV32EIDR, U23 TPS1H000AQDGNRQ1, U24 AM26LV32EIDR, U25 TPS1H000AQDGNRQ1, U26 AM26LV32EIDR, U27 TPS1H000AQDGNRQ1, U28 AM26LV32EIDR, U29 TLP2361, U3 TPS62A02ADRLR, U30 TPS2553DBVR, U31 TPD4E05U06DQAR, U32 TPD4E05U06DQAR, U33 TPD4E05U06DQAR, U34 TPD4E05U06DQAR, U35 TPD4E05U06DQAR, U36 OPA2990IDR, U37 SN74AHCT1G125DBVR, U38 CA-IS3092W, U39 LTV-357T-C, U4 LAN9253-I/R4X, U40 TPS3828-33DBVR, U5 TPS3808G33DBVR, U6 M24C16-RMN6TP, U7 TPD4E05U06DQAR, U8 TPD4E05U06DQAR, U9 STM32H523VET6, X1 SiT8008BI-71-33E-25.000000

Commit message: Supplies done: +VIN trunk to the encoder jumpers, +5V and +VIN fanouts
- Pass "trunk" first: the planes, then a 1 mm +VIN track on layer 4 to the
  four encoder supply jumpers (4 x 0.6 A at most), along the first clear
  corridor above the axes and down the first clear line from the right edge
  to two 0.8/0.4 mm vias in the plane. All or nothing.
- Encoder supply jumpers JP1 to JP4 turned over: +VIN pin up toward the trunk,
  +5V pin down over its plane.
- Passes in order: trunk, gnd, vin, 5v, 3v3, short; the supplies that carry
  current first, the thin links of the later ones route around them.
- A new via keeps its hole 0.25 mm from the tracks of other nets.
- Pass "short" (written, not run yet): pads up to 3 mm apart joined straight.
Parts:
- moved C60 7.79 mm to (11.2, 24.2)
- moved R81 6.32 mm to (13.7, 18.6), turned to -90 degrees
- moved C59 6.05 mm to (10.4, 16.1)
- moved JP1 5.08 mm to (5.70, 24.9), turned to 180 degrees
- moved JP4 5.08 mm to (142.1, 33.8), turned to 180 degrees
- moved JP2 5.08 mm to (79.2, 22.8), turned to 180 degrees
- moved JP3 5.08 mm to (114.7, 26.8), turned to 180 degrees
- moved R89 4.34 mm to (13.5, 26.3), turned to 0 degrees
- moved D22 4.04 mm to (110.8, 18.0), turned to 90 degrees
- moved R73 3.50 mm to (109.7, 22.1), turned to -90 degrees
- moved R72 2.09 mm to (114.8, 15.7)
- moved R90 1.36 mm to (11.4, 20.0), turned to 90 degrees
- moved C66 0.87 mm to (110.8, 25.2), turned to -90 degrees
- moved D16 0.76 mm to (85.7, 24.3), turned to 90 degrees
- moved R75 0.57 mm to (113.3, 30.5), turned to 0 degrees
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Routing:
- net +VIN: track 0.00 -> 333.4 mm, vias 0 -> 19
- net +5V: track 0.00 -> 133.8 mm, vias 0 -> 65
- net +3V3: track 351.1 -> 368.4 mm, vias 122 -> 123

Commit message: Pass short: pads up to 3 mm apart joined on layer 1, straight or with one bend
Routing:
- net /ESC/VDD33TXRX2: track 0.00 -> 14.8 mm
- net /ESC/VDD33TXRX1: track 0.00 -> 9.72 mm
- net Net-(D47-COM): track 0.00 -> 5.93 mm
- net Net-(Q5-E): track 0.00 -> 5.75 mm
- net Net-(D69-A): track 0.00 -> 5.66 mm
- net /Encoder 1/VENC: track 0.00 -> 5.46 mm
- net /MCU/VDDA: track 0.00 -> 5.30 mm
- net SPINDLE_EN: track 0.00 -> 4.75 mm
- net SPINDLE_DIR: track 0.00 -> 4.75 mm
- net Net-(Q11-G): track 0.00 -> 4.75 mm
- net ENA1: track 0.00 -> 4.50 mm
- net Net-(U36-+INA): track 0.00 -> 4.27 mm
- net Net-(U9-PC9): track 0.00 -> 3.75 mm
- net /ESC/RBIAS: track 0.00 -> 3.25 mm
- net Net-(D41-COM): track 0.00 -> 3.00 mm
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