File: hardware/base/kicad/bus.kicad_sch (KiCad schematic)
At the start: 46 parts, among them J15 LOCAL BUS, U30 TPS2553DBVR

Commit message: Harden the base board protections and unify its terminal blocks
- TVS (SMBJ33CA) on the spindle EN and DIR drains: a relay coil driven
  without a flyback diode no longer avalanches the FET.
- ESD (5 x TPD4E05U06) on every signal of the local bus header.
- A single terminal block type, KF2EDGR-3.81-4P, five times. Pinout rule:
  pole 1 withstands 24 V, pole 2 is 0 V, so the power plug damages
  nothing whichever header it lands in.
- Functional earth on pole 3 of the power terminal block, replacing the
  M3 earth lug.
- 100 k pull-down on the DAC node: the 0-10 V output stays at 0 V while
  the DAC pin is not configured (reset, bootloader).
- "24V OUT" LED on +24V_DRV and test points on the four rails.
Parts:
- removed J15: LOCAL BUS, Connector_IDC:IDC-Header_2x17_P2.54mm_Vertical, symbol Connector_Generic:Conn_02x17_Odd_Even
- added J14: LOCAL BUS, Connector_IDC:IDC-Header_2x17_P2.54mm_Vertical, symbol Connector_Generic:Conn_02x17_Odd_Even
- added U31, U32, U33, U34, U35: TPD4E05U06DQAR, Package_SON:USON-10_2.5x1.0mm_P0.5mm, symbol Power_Protection:TPD4E05U06DQA
Connections:
- net +3V3_BUS: now also J14.30 (Pin_30), J14.31 (Pin_31)
- net BUS_IRQ: now also J14.10 (Pin_10), U32.2 (D1-)
- net BUS_MISO: now also J14.5 (Pin_5), U31.4 (D2+)
- net BUS_SCL: now also J14.12 (Pin_12), U32.5 (D2-)
- net BUS_SDA: now also J14.11 (Pin_11), U32.4 (D2+)
- net GND: now also J14.1 (Pin_1), J14.13 (Pin_13), J14.17 (Pin_17), J14.21 (Pin_21), J14.25 (Pin_25), J14.29 (Pin_29), J14.3 (Pin_3), J14.32 (Pin_32), J14.33 (Pin_33), J14.34 (Pin_34), J14.6 (Pin_6), J14.9 (Pin_9), U31.3 (GND), U31.8 (GND), U32.3 (GND), U32.8 (GND), U33.3 (GND), U33.8 (GND), U34.3 (GND), U34.8 (GND), U35.3 (GND), U35.8 (GND)
- net RB_CS0: now also J14.14 (Pin_14), U33.1 (D1+)
- net RB_CS1: now also J14.15 (Pin_15), U33.2 (D1-)
- net RB_CS10: now also J14.27 (Pin_27), U35.4 (D2+)
- net RB_CS11: now also J14.28 (Pin_28), U35.5 (D2-)
- net RB_CS2: now also J14.16 (Pin_16), U33.4 (D2+)
- net RB_CS3: now also J14.18 (Pin_18), U33.5 (D2-)
- net RB_CS4: now also J14.19 (Pin_19), U34.1 (D1+)
- net RB_CS5: now also J14.20 (Pin_20), U34.2 (D1-)
- net RB_CS6: now also J14.22 (Pin_22), U34.4 (D2+)
- net RB_CS7: now also J14.23 (Pin_23), U34.5 (D2-)
- net RB_CS8: now also J14.24 (Pin_24), U35.1 (D1+)
- net RB_CS9: now also J14.26 (Pin_26), U35.2 (D1-)
- net RB_LATCH: now also J14.7 (Pin_7), U31.5 (D2-)
- net RB_MOSI: now also J14.4 (Pin_4), U31.2 (D1-)
- net RB_OE: now also J14.8 (Pin_8), U32.1 (D1+)
- net RB_SCK: now also J14.2 (Pin_2), U31.1 (D1+)
- no-connect marks 0 -> 20
Other:
- note added: "ESD of every ribbon signal at the header (TPD4E05U06, flow-through)."

Commit message: Accept a 12 V or 24 V supply on the base board (10.8 to 30 V)
- Supply nets renamed +VIN and +VIN_OUT (silkscreen VIN OUT).
- UVLO 200 k over 47 k // 100 k: start 8.47 V (9.48 V worst case),
  stop 7.79 V; fuse 3.5 A (12H1350C).
- 0-10 V: OPA2990 rail-to-rail op amp supplied by +VIN, SS8550 current
  limit across the 120 ohm; 10 V into 10 k from 10.9 V of supply.
- E-stop and probe inputs: 2 x 4.7 k in parallel, shunts 1 k and 4.7 k.
- Buck simulated from 7.8 to 30 V with the smallest slope compensation
  the datasheet allows: 79 deg, 11.6 dB minimum.
Parts:
- removed R186: 47k, Resistor_SMD:R_0402_1005Metric, symbol Device:R
- added R227: 2.2k, Resistor_SMD:R_0402_1005Metric, symbol Device:R
- R187: value 1k -> 47k; LCSC C11702 -> C25792
- R188: value 10k -> 1k; LCSC C25744 -> C11702
- R202: value 49.9 -> 10k; LCSC C25120 -> C25744
- R221: value 10k -> 49.9; LCSC C25744 -> C25120
- R222: value 100k -> 10k; LCSC C25741 -> C25744
- R225: value 2.2k -> 100k; LCSC C25879 -> C25741
Connections:
- net +3V3: now also R188.1, R202.2, R222.2, R227.2; no longer R187.1, R188.2, R221.2, R225.2
- net BUS_CS0: now also R189.1, R203.1; no longer R188.1, R202.1
- net BUS_CS1: now also R190.1, R204.1; no longer R189.1, R203.1
- net BUS_CS10: now also R199.1, R213.1; no longer R198.1, R212.1
- net BUS_CS11: now also R200.1, R214.1; no longer R199.1, R213.1
- net BUS_CS2: now also R191.1, R205.1; no longer R190.1, R204.1
- net BUS_CS3: now also R192.1, R206.1; no longer R191.1, R205.1
- net BUS_CS4: now also R193.1, R207.1; no longer R192.1, R206.1
- net BUS_CS5: now also R194.1, R208.1; no longer R193.1, R207.1
- net BUS_CS6: now also R195.1, R209.1; no longer R194.1, R208.1
- net BUS_CS7: now also R196.1, R210.1; no longer R195.1, R209.1
- net BUS_CS8: now also R197.1, R211.1; no longer R196.1, R210.1
- net BUS_CS9: now also R198.1, R212.1; no longer R197.1, R211.1
- net BUS_IRQ: now also R222.1; no longer R221.1
- net BUS_LATCH: now also R201.1, R217.1, R221.1; no longer R200.1, R216.1, R220.1
- net BUS_MISO: now also R223.1; no longer R222.1
- net BUS_MOSI: now also R216.1, R220.1, R225.1; no longer R215.1, R219.1, R224.1
- net BUS_OE: now also R202.1, R218.1; no longer R201.1, R217.1
- net BUS_SCK: now also R215.1, R219.1, R224.1; no longer R214.1, R218.1, R223.1
- net BUS_SCL: now also R227.1; no longer R226.1
- net BUS_SDA: now also R226.1; no longer R225.1
- net GND: now also R187.2, R225.2; no longer R222.2
- net RB_CS0: now also R203.2; no longer R202.2
- net RB_CS1: now also R204.2; no longer R203.2
- net RB_CS10: now also R213.2; no longer R212.2
- net RB_CS11: now also R214.2; no longer R213.2
- net RB_CS2: now also R205.2; no longer R204.2
- net RB_CS3: now also R206.2; no longer R205.2
- net RB_CS4: now also R207.2; no longer R206.2
- net RB_CS5: now also R208.2; no longer R207.2
- net RB_CS6: now also R209.2; no longer R208.2
- net RB_CS7: now also R210.2; no longer R209.2
- net RB_CS8: now also R211.2; no longer R210.2
- net RB_CS9: now also R212.2; no longer R211.2
- net RB_LATCH: now also R217.2, R221.2; no longer R216.2, R220.2
- net RB_MOSI: now also R216.2, R220.2; no longer R215.2, R219.2
- net RB_OE: now also R218.2; no longer R217.2
- net RB_SCK: now also R215.2, R219.2; no longer R214.2, R218.2
- net at D58.2 (A): now also R188.2; no longer R187.2
- net at U30.5 (ILIM): now also R187.1
Other:
- moved on the sheet: R187

Commit message: Start the base board PCB: outline, profile rules, connectors on the edges
- pcb.py builds the board from the schematic: 72 x 150 mm, 4 layers,
  C-LOCK keyhole, M3 holes, connectors on both long edges; the other
  parts are parked beside the board until they are placed.
- base.kicad_dru: rules of the Phoenix UM-BASIC 72 profile (no part at
  the short edges on the top side, no through-hole lead on the rim the
  board rests on), proved by the DRC.
- Dual shielded RJ45 per axis (HC-WK88-H132-1X2-55B): port A for the
  drive, port B for the encoder. kicadgen draws multi-unit symbols, one
  unit per sheet; footprint and 3D model generated from the datasheet.
Parts:
- removed J14: LOCAL BUS, Connector_IDC:IDC-Header_2x17_P2.54mm_Vertical, symbol Connector_Generic:Conn_02x17_Odd_Even
- added J10: LOCAL BUS, Connector_IDC:IDC-Header_2x17_P2.54mm_Vertical, symbol Connector_Generic:Conn_02x17_Odd_Even
Connections:
- net +3V3_BUS: now also J10.30 (Pin_30), J10.31 (Pin_31)
- net BUS_IRQ: now also J10.10 (Pin_10)
- net BUS_MISO: now also J10.5 (Pin_5)
- net BUS_SCL: now also J10.12 (Pin_12)
- net BUS_SDA: now also J10.11 (Pin_11)
- net GND: now also J10.1 (Pin_1), J10.13 (Pin_13), J10.17 (Pin_17), J10.21 (Pin_21), J10.25 (Pin_25), J10.29 (Pin_29), J10.3 (Pin_3), J10.32 (Pin_32), J10.33 (Pin_33), J10.34 (Pin_34), J10.6 (Pin_6), J10.9 (Pin_9)
- net RB_CS0: now also J10.14 (Pin_14)
- net RB_CS1: now also J10.15 (Pin_15)
- net RB_CS10: now also J10.27 (Pin_27)
- net RB_CS11: now also J10.28 (Pin_28)
- net RB_CS2: now also J10.16 (Pin_16)
- net RB_CS3: now also J10.18 (Pin_18)
- net RB_CS4: now also J10.19 (Pin_19)
- net RB_CS5: now also J10.20 (Pin_20)
- net RB_CS6: now also J10.22 (Pin_22)
- net RB_CS7: now also J10.23 (Pin_23)
- net RB_CS8: now also J10.24 (Pin_24)
- net RB_CS9: now also J10.26 (Pin_26)
- net RB_LATCH: now also J10.7 (Pin_7)
- net RB_MOSI: now also J10.4 (Pin_4)
- net RB_OE: now also J10.8 (Pin_8)
- net RB_SCK: now also J10.2 (Pin_2)

Commit message: Differential pairs routed by script; PHY to jack mapping for a planar layout
- pairs.py, pass "pairs" right after the planes and trunks: A* on a 0.1 mm
  grid for the centre line of each pair, clear of the other copper by about
  3 W (by the clearance alone near the pads), offset into its two lines;
  straight out of the QFN pads, straight through the ESD arrays, each line on
  its own into the through-hole pins of the jack. Ethernet 100 ohm and USB
  90 ohm at 0.15 mm gap (sim/impedance.py).
- Schematic: the lines on the jack pins and ESD channels in the order that
  routes without a crossing (port A with P and N swapped, port B with TX and
  RX swapped: the LAN9253 PHYs correct the polarity and have HP Auto-MDIX);
  the NC pins of the ESD arrays opposite each line carry it (TI flow-through).
- Ethernet terminations lifted off the board while the pairs are routed, then
  put against their line, 2 to 10 mm from the PHY pins; the lines inside a
  port straddled by their 0603 termination (49.9 ohm moved to 0603, C23185,
  basic, 1.78 M in stock on 2026-10-20; clock series resistors too).
- Placement: lanes of the pairs kept free of other parts (LAN9253 checklist);
  ESD arrays in the way of their lines; centre tap capacitors at the jacks;
  VDD33TXRX mini-planes in layer 3 under the terminations.
- route.py: real C-LOCK cutout clearance for copper; via hole to pad
  clearance; mini-plane priority in the plane test.
- kicadgen: tagged labels do not name a net (a second label on a NC pin).

Claude-Session: https://claude.ai/code/session_01D6Na26JP4CWdxCU6BKa4Yc
Parts:
- R203, R204, R205, R206, R207, R208, R209, R210, R211, R212, R213, R214, R215, R216, R217, R218, R219, R220, R221: footprint Resistor_SMD:R_0402_1005Metric -> Resistor_SMD:R_0603_1608Metric; LCSC C25120 -> C23185
