File: hardware/base/kicad/bus.kicad_sch (KiCad schematic)
At the start: 51 parts, among them J10 LOCAL BUS, U30 TPS2553DBVR, U31 TPD4E05U06DQAR, U32 TPD4E05U06DQAR, U33 TPD4E05U06DQAR, U34 TPD4E05U06DQAR, U35 TPD4E05U06DQAR

Commit message: Lanes no longer shadowed in the assembly; channel assignments carried; encoder sheet drawn from the wired channels; trunk drop found across the board
Connections:
- net BUS_IRQ: now also U32.1 (D1+); no longer U32.2 (D1-)
- net BUS_SCL: now also U32.4 (D2+); no longer U32.5 (D2-)
- net BUS_SDA: now also U32.5 (D2-); no longer U32.4 (D2+)
- net RB_CS1: now also U33.4 (D2+); no longer U33.2 (D1-)
- net RB_CS2: now also U33.2 (D1-); no longer U33.4 (D2+)
- net RB_OE: now also U32.2 (D1-); no longer U32.1 (D1+)

Commit message: Local bus: chip selects first on consecutive pins, every other line on an even pin facing a ground, board VIN on pins 33-34 behind one 480 mA switch per pin, a ground as its only neighbour
Parts:
- added C313, C316: 100nF, Capacitor_SMD:C_0402_1005Metric, symbol Device:C
- added C314, C315, C317, C318: 1µF 50V, Capacitor_SMD:C_0603_1608Metric, symbol Device:C
- added R312, R314: 10k, Resistor_SMD:R_0402_1005Metric, symbol Device:R
- added R313, R315: 1k, Resistor_SMD:R_0402_1005Metric, symbol Device:R
- added U302, U303: TPS1H000AQDGNRQ1, Package_SO:HVSSOP-8-1EP_3x3mm_P0.65mm_EP1.57x1.89mm, symbol Bornier:TPS1H000
Connections:
- net +3V3: now also R312.2, R314.2, U302.1 (IN), U303.1 (IN)
- net +3V3_BUS: now also J10.14 (Pin_14); no longer J10.30 (Pin_30)
- net BUS_IRQ: now also J10.30 (Pin_30), U35.5 (D2-); no longer J10.10 (Pin_10), U32.1 (D1+)
- net BUS_MISO: now also J10.24 (Pin_24), U35.1 (D1+); no longer J10.5 (Pin_5), U31.4 (D2+)
- net BUS_SCL: now also J10.18 (Pin_18), U34.2 (D1-); no longer J10.12 (Pin_12), U32.4 (D2+)
- net BUS_SDA: now also J10.16 (Pin_16), U34.1 (D1+); no longer J10.11 (Pin_11), U32.5 (D2-)
- net GND: now also J10.15 (Pin_15), J10.19 (Pin_19), J10.23 (Pin_23), J10.27 (Pin_27), C313.2, C314.2, C315.2, C316.2, C317.2, C318.2, R313.2, R315.2, U302.2 (DIAG_EN), U302.6 (GND), U302.9 (EP), U303.2 (DIAG_EN), U303.6 (GND), U303.9 (EP); no longer J10.1 (Pin_1), J10.3 (Pin_3), J10.33 (Pin_33), J10.34 (Pin_34), J10.6 (Pin_6), J10.9 (Pin_9)
- net RB_CS0: now also J10.1 (Pin_1), U31.1 (D1+); no longer J10.14 (Pin_14), U33.1 (D1+)
- net RB_CS1: now also J10.2 (Pin_2), U31.2 (D1-); no longer J10.15 (Pin_15), U33.4 (D2+)
- net RB_CS10: now also J10.11 (Pin_11), U33.4 (D2+); no longer J10.27 (Pin_27), U35.4 (D2+)
- net RB_CS11: now also J10.12 (Pin_12), U33.5 (D2-); no longer J10.28 (Pin_28), U35.5 (D2-)
- net RB_CS2: now also J10.3 (Pin_3), U31.4 (D2+); no longer J10.16 (Pin_16), U33.2 (D1-)
- net RB_CS3: now also J10.4 (Pin_4), U31.5 (D2-); no longer J10.18 (Pin_18), U33.5 (D2-)
- net RB_CS4: now also J10.5 (Pin_5), U32.1 (D1+); no longer J10.19 (Pin_19), U34.1 (D1+)
- net RB_CS5: now also J10.6 (Pin_6), U32.2 (D1-); no longer J10.20 (Pin_20), U34.2 (D1-)
- net RB_CS6: now also J10.7 (Pin_7), U32.4 (D2+); no longer J10.22 (Pin_22), U34.4 (D2+)
- net RB_CS7: now also J10.8 (Pin_8), U32.5 (D2-); no longer J10.23 (Pin_23), U34.5 (D2-)
- net RB_CS8: now also J10.9 (Pin_9), U33.1 (D1+); no longer J10.24 (Pin_24), U35.1 (D1+)
- net RB_CS9: now also J10.10 (Pin_10), U33.2 (D1-); no longer J10.26 (Pin_26), U35.2 (D1-)
- net RB_LATCH: now also J10.26 (Pin_26), U35.2 (D1-); no longer J10.7 (Pin_7), U31.5 (D2-)
- net RB_MOSI: now also J10.22 (Pin_22), U34.5 (D2-); no longer J10.4 (Pin_4), U31.2 (D1-)
- net RB_OE: now also J10.28 (Pin_28), U35.4 (D2+); no longer J10.8 (Pin_8), U32.2 (D1-)
- net RB_SCK: now also J10.20 (Pin_20), U34.4 (D2+); no longer J10.2 (Pin_2), U31.1 (D1+)
- new net: R313.1, U302.4 (CL)
- new net: R312.1, U302.5 (DELAY)
- new net: R314.1, U303.5 (DELAY)
- new net: R315.1, U303.4 (CL)
- new net +VIN: C313.1, C314.1, C316.1, C317.1, U302.8 (VS), U303.8 (VS)
- new net +VIN_BUS1: C315.1, J10.33 (Pin_33), U302.7 (OUT)
- new net +VIN_BUS2: C318.1, J10.34 (Pin_34), U303.7 (OUT)
- no-connect marks 20 -> 22
Other:
- note added: "+VIN_BUS1, +VIN_BUS2: the supply voltage on ribbon pins 33 and 34, one switch per pin, 480 mA limit each, auto-retry."
- note added: "Ribbon: conductor n = pin n. CS0-CS11 on pins 1-12; every other line on an even pin with a ground facing it; VIN_BUS on pins 33-34, its only neighbour a ground (pin 32)."
- note removed: "Ribbon: conductor n = pin n; a ground next to SCK and between groups."

Commit message: Flow-through ESD arrays: the NC pin opposite each protected line carries it on every TPD4E05, not only on the PHY lines
Connections:
- net BUS_IRQ: now also U35.6 (NC)
- net BUS_MISO: now also U35.10 (NC)
- net BUS_SCL: now also U34.9 (NC)
- net BUS_SDA: now also U34.10 (NC)
- net RB_CS0: now also U31.10 (NC)
- net RB_CS1: now also U31.9 (NC)
- net RB_CS10: now also U33.7 (NC)
- net RB_CS11: now also U33.6 (NC)
- net RB_CS2: now also U31.7 (NC)
- net RB_CS3: now also U31.6 (NC)
- net RB_CS4: now also U32.10 (NC)
- net RB_CS5: now also U32.9 (NC)
- net RB_CS6: now also U32.7 (NC)
- net RB_CS7: now also U32.6 (NC)
- net RB_CS8: now also U33.10 (NC)
- net RB_CS9: now also U33.9 (NC)
- net RB_LATCH: now also U35.9 (NC)
- net RB_MOSI: now also U34.6 (NC)
- net RB_OE: now also U35.7 (NC)
- net RB_SCK: now also U34.7 (NC)
- no-connect marks 22 -> 2

Commit message: Base: pin swaps of the placed board (chip selects, step/dir/enable channels, encoder timers 0 and 1, ribbon and Ethernet A ESD channels)
Connections:
- net RB_CS0: now also U31.5 (D2-), U31.6 (NC); no longer U31.1 (D1+), U31.10 (NC)
- net RB_CS10: now also U33.5 (D2-), U33.6 (NC); no longer U33.4 (D2+), U33.7 (NC)
- net RB_CS11: now also U33.4 (D2+), U33.7 (NC); no longer U33.5 (D2-), U33.6 (NC)
- net RB_CS2: now also U31.1 (D1+), U31.10 (NC); no longer U31.4 (D2+), U31.7 (NC)
- net RB_CS3: now also U31.4 (D2+), U31.7 (NC); no longer U31.5 (D2-), U31.6 (NC)
- net RB_CS4: now also U32.4 (D2+), U32.7 (NC); no longer U32.1 (D1+), U32.10 (NC)
- net RB_CS6: now also U32.5 (D2-), U32.6 (NC); no longer U32.4 (D2+), U32.7 (NC)
- net RB_CS7: now also U32.1 (D1+), U32.10 (NC); no longer U32.5 (D2-), U32.6 (NC)
- net RB_CS8: now also U33.2 (D1-), U33.9 (NC); no longer U33.1 (D1+), U33.10 (NC)
- net RB_CS9: now also U33.1 (D1+), U33.10 (NC); no longer U33.2 (D1-), U33.9 (NC)
