File: hardware/base/kicad/clock.kicad_sch (KiCad schematic)
At the start: 4 parts, among them X1 SiT8008BI-71-33E-25.000000

Commit message: Differential pairs routed by script; PHY to jack mapping for a planar layout
- pairs.py, pass "pairs" right after the planes and trunks: A* on a 0.1 mm
  grid for the centre line of each pair, clear of the other copper by about
  3 W (by the clearance alone near the pads), offset into its two lines;
  straight out of the QFN pads, straight through the ESD arrays, each line on
  its own into the through-hole pins of the jack. Ethernet 100 ohm and USB
  90 ohm at 0.15 mm gap (sim/impedance.py).
- Schematic: the lines on the jack pins and ESD channels in the order that
  routes without a crossing (port A with P and N swapped, port B with TX and
  RX swapped: the LAN9253 PHYs correct the polarity and have HP Auto-MDIX);
  the NC pins of the ESD arrays opposite each line carry it (TI flow-through).
- Ethernet terminations lifted off the board while the pairs are routed, then
  put against their line, 2 to 10 mm from the PHY pins; the lines inside a
  port straddled by their 0603 termination (49.9 ohm moved to 0603, C23185,
  basic, 1.78 M in stock on 2026-10-20; clock series resistors too).
- Placement: lanes of the pairs kept free of other parts (LAN9253 checklist);
  ESD arrays in the way of their lines; centre tap capacitors at the jacks;
  VDD33TXRX mini-planes in layer 3 under the terminations.
- route.py: real C-LOCK cutout clearance for copper; via hole to pad
  clearance; mini-plane priority in the plane test.
- kicadgen: tagged labels do not name a net (a second label on a NC pin).

Claude-Session: https://claude.ai/code/session_01D6Na26JP4CWdxCU6BKa4Yc
Parts:
- R15, R16: footprint Resistor_SMD:R_0402_1005Metric -> Resistor_SMD:R_0603_1608Metric; LCSC C25120 -> C23185
