File: hardware/base/kicad/modbus.kicad_sch (KiCad schematic)
At the start: 19 parts, among them J17 MODBUS, U33 CA-IS3092W

Commit message: Harden the base board protections and unify its terminal blocks
- TVS (SMBJ33CA) on the spindle EN and DIR drains: a relay coil driven
  without a flyback diode no longer avalanches the FET.
- ESD (5 x TPD4E05U06) on every signal of the local bus header.
- A single terminal block type, KF2EDGR-3.81-4P, five times. Pinout rule:
  pole 1 withstands 24 V, pole 2 is 0 V, so the power plug damages
  nothing whichever header it lands in.
- Functional earth on pole 3 of the power terminal block, replacing the
  M3 earth lug.
- 100 k pull-down on the DAC node: the 0-10 V output stays at 0 V while
  the DAC pin is not configured (reset, bootloader).
- "24V OUT" LED on +24V_DRV and test points on the four rails.
Parts:
- removed D65: PSM712-LF-T7, Package_TO_SOT_SMD:SOT-23, symbol Diode:SM712_SOT23
- removed D66: green TX, LED_SMD:LED_0603_1608Metric, symbol Device:LED
- removed R241: 10k, Resistor_SMD:R_0402_1005Metric, symbol Device:R
- removed U33: CA-IS3092W, Package_SO:SOIC-16W_7.5x10.3mm_P1.27mm, symbol Bornier:CA-IS3092W
- added D68: green TX, LED_SMD:LED_0603_1608Metric, symbol Device:LED
- added D69: green RX, LED_SMD:LED_0603_1608Metric, symbol Device:LED
- added R249: 1k, Resistor_SMD:R_0402_1005Metric, symbol Device:R
- added U38: CA-IS3092W, Package_SO:SOIC-16W_7.5x10.3mm_P1.27mm, symbol Bornier:CA-IS3092W
- D67: value green RX -> PSM712-LF-T7; footprint LED_SMD:LED_0603_1608Metric -> Package_TO_SOT_SMD:SOT-23; symbol Device:LED -> Diode:SM712_SOT23; LCSC C2289 -> C32677
- R242: value 120 -> 10k; footprint Resistor_SMD:R_0603_1608Metric -> Resistor_SMD:R_0402_1005Metric; LCSC C22787 -> C25744
- R247: value 1k -> 120; footprint Resistor_SMD:R_0402_1005Metric -> Resistor_SMD:R_0603_1608Metric; LCSC C11702 -> C22787
Connections:
- net +3V3: now also R249.1, U38.1 (VCC); no longer R247.1
- net CHASSIS: now also J17.1 (Pin_1); no longer J17.4 (Pin_4)
- net GND: now also R242.2, U38.2 (GNDA), U38.4 (~{RE}), U38.7 (GNDA), U38.8 (GNDA)
- net GNDISO: now also D67.3 (common), J17.2 (Pin_2), R246.2, U38.10 (SEL), U38.15 (GNDB), U38.9 (GNDB); no longer J17.3 (Pin_3), R245.2
- net MB_A: now also D67.1 (A1), J17.3 (Pin_3), R244.2, R247.1, U38.12 (A); no longer J17.1 (Pin_1), R243.2, R246.1
- net MB_B: now also D67.2 (A2), J17.4 (Pin_4), R245.1, U38.13 (B); no longer J17.2 (Pin_2), R244.1
- net MB_DE: now also R242.1, U38.5 (DE)
- net MB_RX: now also D69.1 (K), U38.3 (RO); no longer D67.1 (K)
- net MB_TX: now also D68.1 (K), U38.6 (DI)
- net VISO: now also R243.1, U38.16 (VISO); no longer R242.1
- net at R247.2: now also JP17.1 (A)
- net at R248.2: now also D68.2 (A); no longer D67.2 (A)
- new net: R245.2, R246.1
- new net: R243.2, R244.1
- new net: D69.2 (A), R249.2
Other:
- moved on the sheet: C85, J17, R242, R243, R244, R245, R246, R247, R248

Commit message: Accept a 12 V or 24 V supply on the base board (10.8 to 30 V)
- Supply nets renamed +VIN and +VIN_OUT (silkscreen VIN OUT).
- UVLO 200 k over 47 k // 100 k: start 8.47 V (9.48 V worst case),
  stop 7.79 V; fuse 3.5 A (12H1350C).
- 0-10 V: OPA2990 rail-to-rail op amp supplied by +VIN, SS8550 current
  limit across the 120 ohm; 10 V into 10 k from 10.9 V of supply.
- E-stop and probe inputs: 2 x 4.7 k in parallel, shunts 1 k and 4.7 k.
- Buck simulated from 7.8 to 30 V with the smallest slope compensation
  the datasheet allows: 79 deg, 11.6 dB minimum.
Parts:
- removed C81: 100nF, Capacitor_SMD:C_0402_1005Metric, symbol Device:C
- removed D69: green RX, LED_SMD:LED_0603_1608Metric, symbol Device:LED
- removed R249: 1k, Resistor_SMD:R_0402_1005Metric, symbol Device:R
- added C86: 1nF 2kV, Capacitor_SMD:C_1206_3216Metric, symbol Device:C
- added D66: PSM712-LF-T7, Package_TO_SOT_SMD:SOT-23, symbol Diode:SM712_SOT23
- added R241: 10k, Resistor_SMD:R_0402_1005Metric, symbol Device:R
- C82, C84: value 10µF 25V -> 100nF; footprint Capacitor_SMD:C_0805_2012Metric -> Capacitor_SMD:C_0402_1005Metric; LCSC C15850 -> C307331
- C83: value 100nF -> 10µF 25V; footprint Capacitor_SMD:C_0402_1005Metric -> Capacitor_SMD:C_0805_2012Metric; LCSC C307331 -> C15850
- C85: value 1nF 2kV -> 10µF 25V; footprint Capacitor_SMD:C_1206_3216Metric -> Capacitor_SMD:C_0805_2012Metric; LCSC C9196 -> C15850
- D67: value PSM712-LF-T7 -> green TX; footprint Package_TO_SOT_SMD:SOT-23 -> LED_SMD:LED_0603_1608Metric; symbol Diode:SM712_SOT23 -> Device:LED; LCSC C32677 -> C2289
- D68: value green TX -> green RX
- R242: value 10k -> 120; footprint Resistor_SMD:R_0402_1005Metric -> Resistor_SMD:R_0603_1608Metric; LCSC C25744 -> C22787
- R247: value 120 -> 1k; footprint Resistor_SMD:R_0603_1608Metric -> Resistor_SMD:R_0402_1005Metric; LCSC C22787 -> C11702
Connections:
- net +3V3: now also C83.1, R247.1
- net CHASSIS: now also C86.2; no longer C85.2
- net GND: now also C83.2, R241.2; no longer R242.2
- net GNDISO: now also C85.2, R245.2, C86.1, D66.3 (common); no longer C83.2, C85.1, D67.3 (common), R246.2
- net MB_A: now also R243.2, R246.1, D66.1 (A1); no longer D67.1 (A1), R244.2, R247.1
- net MB_B: now also R244.1, D66.2 (A2); no longer D67.2 (A2), R245.1
- net MB_DE: now also R241.1; no longer R242.1
- net MB_RX: now also D68.1 (K)
- net MB_TX: now also D67.1 (K); no longer D68.1 (K)
- net VISO: now also C85.1, R242.1; no longer C83.1, R243.1
- net at R247.2: now also D67.2 (A); no longer JP17.1 (A)
- new net: R244.2, R245.1
- new net: R242.2, R243.1
- new net: JP17.1 (A), R246.2
Other:
- moved on the sheet: C82, C83, C84, C85, D68, R242, R243, R244, R245, R246, R247, R248

Commit message: Start the base board PCB: outline, profile rules, connectors on the edges
- pcb.py builds the board from the schematic: 72 x 150 mm, 4 layers,
  C-LOCK keyhole, M3 holes, connectors on both long edges; the other
  parts are parked beside the board until they are placed.
- base.kicad_dru: rules of the Phoenix UM-BASIC 72 profile (no part at
  the short edges on the top side, no through-hole lead on the rim the
  board rests on), proved by the DRC.
- Dual shielded RJ45 per axis (HC-WK88-H132-1X2-55B): port A for the
  drive, port B for the encoder. kicadgen draws multi-unit symbols, one
  unit per sheet; footprint and 3D model generated from the datasheet.
Parts:
- removed J17: MODBUS, Connector_Phoenix_MC:PhoenixContact_MC_1,5_4-G-3.81_1x04_P3.81mm_Horizontal, symbol Connector:Screw_Terminal_01x04
- added J13: MODBUS, Connector_Phoenix_MC:PhoenixContact_MC_1,5_4-G-3.81_1x04_P3.81mm_Horizontal, symbol Connector:Screw_Terminal_01x04
Connections:
- net CHASSIS: now also J13.1 (Pin_1)
- net GNDISO: now also J13.2 (Pin_2)
- net MB_A: now also J13.3 (Pin_3)
- net MB_B: now also J13.4 (Pin_4)

Commit message: Place the base board parts; DIP switches for the encoder terminations
Placement (gen/pcb.py): one zone per schematic sheet, key parts placed by
hand, the other parts next to the pin they serve, bulkiest first, with a
1 mm gap preferred when it costs at most 2 mm. The local bus header stands
at the left end, centred across the board, facing the modules.

Encoder terminations: one CTS 218-4LPSTR DIP switch per encoder (100 mA
non-switching) replaces three SMD jumpers; the supply selector and the
Modbus termination use a through-hole 1x3 header. Split DIP symbol, one
unit per switch, drawn on the pair it serves.

DRC rules: 0.2 mm thermal vias, per-package clearance for 0.65 mm pitch
parts. Test points out of the BOM, DNP copied to the footprints. pcb.py
keeps the schematic settings of the project file and finds the KiCad
footprint libraries on every install.

Claude-Session: https://claude.ai/code/session_01JfmMsHNpEd1mfzHNWc4koJ
Parts:
- removed JP17: TERM, Bornier:PinHeader_1x03_P2.54mm_Vertical_SMD_HX_PZ254, symbol Jumper:Jumper_3_Open
- added JP5: TERM, Connector_PinHeader_2.54mm:PinHeader_1x03_P2.54mm_Vertical, symbol Jumper:Jumper_3_Open
Connections:
- net MB_B: now also JP5.2 (C)
- net at R246.2: now also JP5.1 (A)
