File: hardware/base/kicad/modbus.kicad_sch (KiCad schematic)
At the start: 19 parts, among them J13 MODBUS, U38 CA-IS3092W

Commit message: Modbus termination always fitted (R246, removed for a master in the middle of the line); no ESD array on NRST; Ethernet line nets named TXA_P/TXA_N so that tools pair them
Parts:
- removed JP5: TERM, Connector_PinHeader_2.54mm:PinHeader_1x03_P2.54mm_Vertical, symbol Jumper:Jumper_3_Open
Connections:
- net MB_B: now also R246.2
- no-connect marks 3 -> 2
Other:
- note added: "Isolated half-duplex RS-485: the bus side is powered by the DC-DC inside the transceiver (VISO = 3.3 V). Bornier is the master of the line, so it biases it: 370 mV at idle with a 120 ohm termination at each end. Termination always fitted (Bornier at an end of the line); a master in the middle: remove it. Wiring: D1 (A), D0 (B), common, shield."
- note removed: "Isolated half-duplex RS-485: the bus side is powered by the DC-DC inside the transceiver (VISO = 3.3 V). Bornier is the master of the line, so it biases it: 370 mV at idle with a 120 ohm termination at each end. TERM: shunt on 1-2 when Bornier sits at an end of the line. Wiring: D1 (A), D0 (B), common, shield."
- moved on the sheet: R246
