File: hardware/base/kicad/drive.kicad_sch (KiCad schematic)
At the start: 30 parts, among them J6 HC-WK88-H132-1X2-55B, J7 HC-WK88-H132-1X2-55B, Q1 AO3422, Q2 AO3422, U11 ST26C31BDR, U12 LTV-357T-C, U13 TPD4E05U06DQAR, U14 LTV-357T-C, U15 TPD4E05U06DQAR

Commit message: One drive sheet per axis with its own dual RS-422 driver; one placement score for every step, block refinement, cost breakdown by block
Parts:
- removed D16: green ENA, LED_SMD:LED_0603_1608Metric, symbol Device:LED
- removed D17: SMBJ33CA, Diode_SMD:D_SMB, symbol Device:D_TVS
- removed D18: red ALM, LED_SMD:LED_0603_1608Metric, symbol Device:LED
- removed D19: 1N4148WS, Diode_SMD:D_SOD-323, symbol Device:D
- removed J7: HC-WK88-H132-1X2-55B, Bornier:RJ45x2_HongCheng_HC-WK88-H132-1X2-55B, symbol Bornier:RJ45x2_Shielded
- removed Q2: AO3422, Package_TO_SOT_SMD:SOT-23, symbol Transistor_FET:AO3400A
- removed R62, R63, R67: 10k, Resistor_SMD:R_0402_1005Metric, symbol Device:R
- removed R64: 100k, Resistor_SMD:R_0402_1005Metric, symbol Device:R
- removed R65: 1k, Resistor_SMD:R_0402_1005Metric, symbol Device:R
- removed R66: 4.7k, Resistor_SMD:R_1206_3216Metric, symbol Device:R
- removed U14: LTV-357T-C, Package_SO:SO-4_4.4x3.6mm_P2.54mm, symbol Isolator:LTV-357T
- removed U15: TPD4E05U06DQAR, Package_SON:USON-10_2.5x1.0mm_P0.5mm, symbol Power_Protection:TPD4E05U06DQA
- U11: value ST26C31BDR -> SN75ALS191DR; footprint Package_SO:SOIC-16_3.9x9.9mm_P1.27mm -> Package_SO:SOIC-8_3.9x4.9mm_P1.27mm; symbol Interface:AM26LS31CD -> Bornier:SN75ALS191; LCSC C94192 -> C2871261
Connections:
- net +5V: now also U11.1 (VCC); no longer U11.16 (VDD), U11.4 (G)
- net GND: now also U11.4 (GND); no longer U11.12 (~{G}), U11.8 (GND)
- net ALM_A renamed ALM
- net ALM_A_IN renamed ALM_IN
- net DIR_A renamed DIR
- net DIR: now also U11.3 (2A); no longer U11.7 (2A)
- net DIR_A_N renamed DIR_N
- net DIR_A_P renamed DIR_P
- removed net DIR_B: U11.15 (4A)
- removed net DIR_B_N: U11.13 (4Z)
- removed net DIR_B_P: U11.14 (4Y)
- net ENA_A renamed ENA
- net ENA_A_OUT renamed ENA_OUT
- net STEP_A renamed STEP
- net STEP: now also U11.2 (1A); no longer U11.1 (1A)
- net STEP_A_N renamed STEP_N
- net STEP_N: now also U11.7 (1Z); no longer U11.3 (1Z)
- net STEP_A_P renamed STEP_P
- net STEP_P: now also U11.8 (1Y); no longer U11.2 (1Y)
- removed net STEP_B: U11.9 (3A)
- removed net STEP_B_N: U11.11 (3Z)
- removed net STEP_B_P: U11.10 (3Y)
- no-connect marks 8 -> 4
Other:
- note added: "DRIVE PORT"
- note added: "Placed four times: axes 0 to 3. RS-422 STEP/DIR (5 V), ENA open drain to 0 V, ALM through an optocoupler fed by +VIN_OUT. Wiring of a drive: COM+ of its inputs on +VIN_OUT (pin 7), servo-on on ENA (pin 4), its floating alarm output between ALM (pin 5) and 0 V (pin 8)."
- note removed: "DRIVE A"
- note removed: "DRIVE B"
- note removed: "PAIR OF DRIVE PORTS"
- note removed: "Placed twice: axes 0-1 and 2-3 (axis A = even, B = odd). RS-422 STEP/DIR (5 V), ENA open drain to 0 V, ALM through an optocoupler fed by +VIN_OUT. Wiring of a drive: COM+ of its inputs on +VIN_OUT (pin 7), servo-on on ENA (pin 4), its floating alarm output between ALM (pin 5) and 0 V (pin 8)."
- title: Pair of drive ports: STEP/DIR, ENA, ALM (2 instances) -> Drive port: STEP/DIR, ENA, ALM (4 instances)
- moved on the sheet: C56, D12, D13, D14, D15, J6A, Q1, R56, R57, R58, R59, R60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
Changed lines of the file:
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@@
 	(paper "A3")
 	(title_block
-		(title "Pair of drive ports: STEP/DIR, ENA, ALM (2 instances)")
+		(title "Drive port: STEP/DIR, ENA, ALM (4 instances)")
 		(date "2026-10-18")
 		(rev "A")

Commit message: Flow-through ESD arrays: the NC pin opposite each protected line carries it on every TPD4E05, not only on the PHY lines
Connections:
- net DIR_N: now also U13.6 (NC)
- net DIR_P: now also U13.7 (NC)
- net STEP_N: now also U13.9 (NC)
- net STEP_P: now also U13.10 (NC)
- no-connect marks 4 -> 0
